File: gordian-knot.sch (EAGLE design)
At the start: 24 parts, among them J2 PJRAN1X1U01X, J3 PJRAN1X1U01X, J5 PJRAN1X1U01X, J7 PJRAN1X1U01X

Commit message: Add files via upload
Parts:
- removed C1, C2, C3, C4: (no value), adafruit:C-US025-040X050
- removed J1, J4, J6, J8: (no value), Wurth_Elektronik_Electromechanic_Coaxial _Connectors_rev18a:60314002124524
- removed J2, J3, J5, J7: PJRAN1X1U01X, Connectors:PJRAN1X1U01X
- added JP10: (no value), adafruit:PINHD-1X1-BIGPOGO
- added LED1, LED2, LED3, LED4: WS2812B5050, adafruit:WS2812B5050
- added R5: 1K, adafruit:R-US_0207/9
- R1, R2, R3, R4: value (none) -> 1K
Connections:
- removed net N$5: J3.2, R2.1
- removed net N$6: J4.1, JP4.1
- removed net N$7: C3.1, JP5.1, R3.2
- removed net N$8: J5.2, R3.1
- new net VCC: LED1.VDD, LED2.VDD, LED3.VDD, LED4.VDD, R1.2
- net GND: now also LED1.GND, LED2.GND, LED3.GND, LED4.GND, R5.1; no longer C1.2, C2.2, C3.2, C4.2, J1.2, J2.1, J2.3, J3.1, J3.3, J4.2, J5.1, J5.3, J6.2, J7.1, J7.3, J8.2
- net N$1: now also JP2.1, R1.1, R2.2; no longer C1.1, JP1.1, R1.2
- net N$10: now also LED2.DI, LED3.DO; no longer C4.1, JP7.1, R4.2
- net N$11: now also LED3.DI, LED4.DO; no longer J7.2, R4.1
- net N$12: now also JP10.1, LED1.DO; no longer J8.1, JP8.1
- net N$2: now also JP4.1, R2.1, R3.2; no longer J2.2, R1.1
- net N$3: now also JP6.1, R3.1, R4.2; no longer J1.1, JP2.1
- net N$4: now also JP8.1, R4.1, R5.2; no longer C2.1, JP3.1, R2.2
- net N$9: now also LED1.DI, LED2.DO; no longer J6.1, JP6.1
Other:
- note added: "Blue"
- note added: "D7"
- note added: "Green"
- note added: "Red"
- note added: "V2"
- note added: "Yellow"
- note removed: "PWM pin 10"
- note removed: "PWM pin 11"
- note removed: "PWM pin 6"
- note removed: "PWM pin 9"
- moved on the sheet: R1, R2, R3, R4
